File: schema/airsens_v3_0.kicad_sch (KiCad schematic)
At the start: 29 parts, among them J1 ALIM, J3 USB TO UART, U1 MAX604, U2 ESP32-WROOM-32, j2 BME280

Commit message: Add files via upload
Parts:
- added D1: LED, symbol Device:LED
- added J4: PAIR, symbol Connector:Conn_01x01_Male
- added J5: LED, symbol Connector:Conn_01x01_Male
- added LED, PAIR: EN, symbol Connector:Conn_01x01_Female
- added R4: 1k, symbol Device:R
- added U3: PAIR-IO12, Package_SO:SOIC-8_3.9x4.9mm_P1.27mm, symbol Analog_Switch:ADG417BR
- C3: value 1uF -> 10uF
Connections:
- net GND: now also R4.2, U3.
- net at U2.13 (IO14): now also J4.1 (Pin_1)
- net at U2.14 (IO12): now also J5.1 (Pin_1)
- new net: D1.1 (K), R4.1
- new net: D1.2 (A), LED.1 (Pin_1)
- new net: PAIR.1 (Pin_1), U3.
Other:
- moved on the sheet: 3.7V, BOOT, C1, C2, C3, EN, R1, R2, R3, U1, VDD

Commit message: Ready for the hardware
Parts:
- removed J1: ALIM, symbol Connector_Generic:Conn_01x02
- removed J?: UBAT, symbol Connector:Conn_01x01_Male
- removed J?: UBAT, symbol Connector:Conn_01x01_Female
- removed LED: EN, symbol Connector:Conn_01x01_Female
- removed j2: BME280, symbol Connector_Generic:Conn_01x04
- added LED(pin14): EN, symbol Connector:Conn_01x01_Female
- C2: value 10uF -> 1uF
- J?: value ADC_IN -> ADC_IN(pin7)
- U3: value PAIR-IO12 -> PAIR-IO14
- renumbered BOOT to BOOT(pin25), EN to EN(pin3), PAIR to PAIR(pin13), VDD to VDD(pin2)
Connections:
- net at 3.7V.1 (+): now also R1.1, U1.1 (IN), U1.4 (~{OFF})
- net at D1.2 (A): now also LED(pin14).1 (Pin_1)
Other:
- moved on the sheet: 3.7V, BOOT(pin25), C1, C2, C3, EN(pin3), J3, PAIR(pin13), R1, R2, R3, U1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
